File: display.kicad_sch (KiCad schematic)
At the start: 19 parts, among them Q2 AP2302B

Commit message: Fill out all component LCSC numbers and fix footprint associations
Parts:
- C36: LCSC C69335 -> (none); LCSC Part (none) -> C69335
- C37, C38, C39, C41, C42, C43, C44: LCSC C5199872 -> (none); LCSC Part (none) -> C5199872
- C40: LCSC C15849 -> (none); LCSC Part (none) -> C15849
- C45: LCSC C1623 -> (none); LCSC Part (none) -> C1623
- D3, D5, D8: LCSC C22466873 -> (none); LCSC Part (none) -> C22466873
- FPC1: LCSC C22380687 -> (none)
- L9: LCSC C83083 -> (none); LCSC Part (none) -> C83083
- Q2: LCSC C406812 -> (none); LCSC Part (none) -> C406812
- R11: LCSC C2907304 -> (none); LCSC Part (none) -> C2907304
- R12: LCSC C25741 -> (none); LCSC Part (none) -> C25741
- R13: LCSC Part (none) -> -
Connections:
- net 3V3: no longer C36.2, FPC1.10, FPC1.9, R13.1
- new net +3.3V: C36.2, FPC1.10, FPC1.9, R13.1
