File: hackerhotel2027.kicad_pcb (KiCad board)
At the start: 6 copper layers, 95.4 x 99.9 mm, 371 parts, among them J1 USB device, J2 Battery, J3 Debug, Q1 JSM2301S, SW1 TS-1187A-B-A-B, SW2 TS-1187A-B-A-B, SW3 TS-1187A-B-A-B, SW4 TS-1187A-B-A-B, U1 CH643Q, U2 TPD4E05U06DQAR, U3 XT4054K421MR-G

Commit message: Prototype 1
Parts:
- added C7: 10u, Capacitor_SMD:C_0603_1608Metric, B.Cu at (-20.6, 16.7)
- added C8: 1u, Capacitor_SMD:C_0603_1608Metric, B.Cu at (-22.1, 16.7)
- C3: value 10uF -> 10u
- D1, D10, D100, D101, D102, D103, D104, D105, D106, D107, D108, D109, D11, D110, D111, D112, D113, D114, D115, D116, D117, D118, D119, D12, D120, D121, D122, D123, D124, D125, D126, D127, D128, D129, D13, D130, D131, D132, D133, D134, D135, D136, D137, D138, D139, D14, D140, D141, D142, D143, D144, D145, D146, D147, D148, D149, D15, D150, D158, D159, D16, D160, D161, D162, D163, D164, D165, D166, D167, D168, D169, D17, D170, D171, D172, D173, D174, D175, D176, D177, D178, D179, D18, D180, D181, D182, D183, D184, D185, D186, D187, D188, D189, D19, D190, D191, D192, D193, D194, D195, D196, D197, D198, D199, D2, D20, D200, D201, D202, D203, D204, D205, D206, D207, D208, D21, D216, D217, D218, D219, D22, D220, D221, D222, D223, D224, D225, D226, D227, D228, D229, D23, D230, D231, D232, D233, D234, D235, D236, D237, D238, D239, D24, D240, D241, D242, D243, D244, D245, D246, D247, D248, D249, D25, D250, D251, D252, D253, D254, D255, D256, D257, D258, D259, D26, D260, D261, D262, D263, D264, D265, D266, D27, D274, D275, D276, D277, D278, D279, D28, D280, D281, D282, D283, D284, D285, D286, D287, D288, D289, D29, D290, D291, D292, D293, D294, D295, D296, D297, D298, D299, D3, D30, D300, D301, D302, D303, D304, D305, D306, D307, D308, D309, D31, D310, D311, D312, D313, D314, D32, D33, D34, D4, D42, D43, D44, D45, D46, D47, D48, D49, D5, D50, D51, D52, D53, D54, D55, D56, D57, D58, D59, D6, D60, D61, D62, D63, D64, D65, D66, D67, D68, D69, D7, D70, D71, D72, D73, D74, D75, D76, D77, D78, D79, D8, D80, D81, D82, D83, D84, D85, D86, D87, D88, D89, D9, D90, D91, D92: footprint LED_SMD:LED_0402_1005Metric -> led_no_silk:LED_0402_1005Metric_nosilk
- R1, R10, R11, R12, R13, R14, R15, R16, R17, R18, R19, R2, R20, R21, R22, R23, R24, R3, R4, R5, R6, R7, R8, R9: value R -> 200
Routing:
- net R12: track 25.9 -> 22.1 mm
- net VCC: track 19.6 -> 23.0 mm
- net R13: track 27.2 -> 24.3 mm
- net R15: track 29.9 -> 27.1 mm
- net R14: track 28.3 -> 25.5 mm
- net GND: track 37.7 -> 39.9 mm
- net IR_LED: track 62.2 -> 64.1 mm
- net BTN1: track 50.6 -> 52.0 mm
- net /R2b: track 234.9 -> 233.6 mm
- net R10: track 19.7 -> 18.4 mm
- net C10: track 127.1 -> 128.4 mm
- net /R22b: track 135.7 -> 136.7 mm
- net /R24b: track 123.5 -> 122.8 mm
- net R9: track 23.6 -> 22.9 mm
- net USB_DP: track 46.0 -> 46.6 mm
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